Commit message: Adding ot2 alpha and betha into launch file

File: ot2_description/urdf/OT2_robot.xacro (robot description, xacro)
@@ -1,13 +1,25 @@
 <?xml version="1.0"?>
-<robot name="Sealer_Robot" xmlns:xacro="http://www.ros.org/wiki/xacro">
+<robot name="OT2_Robot" xmlns:xacro="http://www.ros.org/wiki/xacro">
   <!-- Materials -->
-  <material name="white">
-    <color rgba="1 1 1 1"/>
-  </material>
-  <material name="aluminum">
-    <color rgba="0.6 0.6 0.6 1"/>
-  </material>
+  <xacro:include filename="$(find ot2_description)/urdf/materials.xacro" />
+  <!-- Module Carts -->
+  <xacro:include filename="$(find ot2_description)/urdf/module_carts.urdf.xacro" />
+  <xacro:Module_Carts prefix="module_carts/"/>
   <!-- OT2 -->
   <xacro:include filename="$(find ot2_description)/urdf/OT2.urdf.xacro" />
   <xacro:OT2 prefix="ot2/"/>
+  <joint name="OT2_alpha" type="fixed">
+    <parent link="module_carts/cart_8"/>
+    <child link="ot2/OT2_alpha"/>
+    <axis xyz="0 0 0"/>
+    <origin xyz="0.825 0.47 0" rpy="0 0 3.1416"/>
+    <limit effort="1000.0" lower="0" upper="0" velocity="0.5"/>
+  </joint>
+  <joint name="OT2_betha" type="fixed">
+    <parent link="module_carts/cart_7"/>
+    <child link="ot2/OT2_betha"/>
+    <axis xyz="0 0 0"/>
+    <origin xyz="0.825 0.47 0" rpy="0 0 3.1416"/>
+    <limit effort="1000.0" lower="0" upper="0" velocity="0.5"/>
+  </joint>
 </robot>

Commit message: Changing robot carts

File: ot2_description/urdf/OT2_robot.xacro (robot description, xacro)
@@ -10,5 +10,5 @@
   <xacro:OT2 prefix="ot2/"/>
   <joint name="OT2_alpha" type="fixed">
-    <parent link="module_carts/cart_8"/>
+    <parent link="module_carts/cart_1"/>
     <child link="ot2/OT2_alpha"/>
     <axis xyz="0 0 0"/>
@@ -17,5 +17,5 @@
   </joint>
   <joint name="OT2_betha" type="fixed">
-    <parent link="module_carts/cart_7"/>
+    <parent link="module_carts/cart_2"/>
     <child link="ot2/OT2_betha"/>
     <axis xyz="0 0 0"/>
@@ -24,5 +24,5 @@
   </joint>
   <joint name="OT2_gamma" type="fixed">
-    <parent link="module_carts/cart_4"/>
+    <parent link="module_carts/cart_5"/>
     <child link="ot2/OT2_gamma"/>
     <axis xyz="0 0 0"/>
