Commit message: Removing extra carts

File: ot2_description/urdf/module_carts.urdf.xacro (robot description, xacro)
@@ -3,9 +3,9 @@
   <!-- Links -->
   <xacro:macro name="Module_Carts" params = "prefix">
-  <link name="${prefix}cart_1">
+  <link name="${prefix}cart_8">
     <visual>
       <origin xyz="0 0 0" rpy="0 0 0"/>
       <geometry>
-        <mesh filename="package://pf400_description/meshes/module_cart.stl" scale="1 1 1"/>
+        <mesh filename="package://ot2_description/meshes/module_cart.stl" scale="1 1 1"/>
       </geometry>
       <material name="darkbluegreen"/>
@@ -13,80 +13,5 @@
     <collision>
       <geometry>
-        <mesh filename="package://pf400_description/meshes/module_cart.stl" scale="1 1 1"/>
-      </geometry>
-      <origin xyz="0 0 0" rpy="0 0 0"/>
-    </collision>
-  </link>
-  <link name="${prefix}cart_2">
-    <visual>
-      <origin xyz="0 0 0" rpy="0 0 0"/>
-      <geometry>
-        <mesh filename="package://pf400_description/meshes/module_cart.stl" scale="1 1 1"/>
-      </geometry>
-      <material name="darkbluegreen"/>
-    </visual>
-    <collision>
-      <geometry>
-        <mesh filename="package://pf400_description/meshes/module_cart.stl" scale="1 1 1"/>
-      </geometry>
-      <origin xyz="0 0 0" rpy="0 0 0"/>
-    </collision>
-  </link>
-  <link name="${prefix}cart_3">
-    <visual>
-      <origin xyz="0 0 0" rpy="0 0 0"/>
-      <geometry>
-        <mesh filename="package://pf400_description/meshes/module_cart.stl" scale="1 1 1"/>
-      </geometry>
-      <material name="darkbluegreen"/>
-    </visual>
-    <collision>
-      <geometry>
-        <mesh filename="package://pf400_description/meshes/module_cart.stl" scale="1 1 1"/>
-      </geometry>
-      <origin xyz="0 0 0" rpy="0 0 0"/>
-    </collision>
-  </link>
-  <link name="${prefix}cart_4">
-    <visual>
-      <origin xyz="0 0 0" rpy="0 0 0"/>
-      <geometry>
-        <mesh filename="package://pf400_description/meshes/module_cart.stl" scale="1 1 1"/>
-      </geometry>
-      <material name="darkbluegreen"/>
-    </visual>
-    <collision>
-      <geometry>
-        <mesh filename="package://pf400_description/meshes/module_cart.stl" scale="1 1 1"/>
-      </geometry>
-      <origin xyz="0 0 0" rpy="0 0 0"/>
-    </collision>
-  </link>
-  <link name="${prefix}cart_5">
-    <visual>
-      <origin xyz="0 0 0" rpy="0 0 0"/>
-      <geometry>
-        <mesh filename="package://pf400_description/meshes/module_cart.stl" scale="1 1 1"/>
-      </geometry>
-      <material name="darkbluegreen"/>
-    </visual>
-    <collision>
-      <geometry>
-        <mesh filename="package://pf400_description/meshes/module_cart.stl" scale="1 1 1"/>
-      </geometry>
-      <origin xyz="0 0 0" rpy="0 0 0"/>
-    </collision>
-  </link>
-  <link name="${prefix}cart_6">
-    <visual>
-      <origin xyz="0 0 0" rpy="0 0 0"/>
-      <geometry>
-        <mesh filename="package://pf400_description/meshes/module_cart.stl" scale="1 1 1"/>
-      </geometry>
-      <material name="darkbluegreen"/>
-    </visual>
-    <collision>
-      <geometry>
-        <mesh filename="package://pf400_description/meshes/module_cart.stl" scale="1 1 1"/>
+        <mesh filename="package://ot2_description/meshes/module_cart.stl" scale="1 1 1"/>
       </geometry>
       <origin xyz="0 0 0" rpy="0 0 0"/>
@@ -97,5 +22,5 @@
       <origin xyz="0 0 0" rpy="0 0 0"/>
       <geometry>
-        <mesh filename="package://pf400_description/meshes/module_cart.stl" scale="1 1 1"/>
+        <mesh filename="package://ot2_description/meshes/module_cart.stl" scale="1 1 1"/>
       </geometry>
       <material name="darkbluegreen"/>
@@ -103,14 +28,14 @@
     <collision>
       <geometry>
-        <mesh filename="package://pf400_description/meshes/module_cart.stl" scale="1 1 1"/>
+        <mesh filename="package://ot2_description/meshes/module_cart.stl" scale="1 1 1"/>
       </geometry>
       <origin xyz="0 0 0" rpy="0 0 0"/>
     </collision>
   </link>
-  <link name="${prefix}cart_8">
+   <link name="${prefix}cart_4">
     <visual>
       <origin xyz="0 0 0" rpy="0 0 0"/>
       <geometry>
-        <mesh filename="package://pf400_description/meshes/module_cart.stl" scale="1 1 1"/>
+        <mesh filename="package://ot2_description/meshes/module_cart.stl" scale="1 1 1"/>
       </geometry>
       <material name="darkbluegreen"/>
@@ -118,81 +43,10 @@
     <collision>
       <geometry>
-        <mesh filename="package://pf400_description/meshes/module_cart.stl" scale="1 1 1"/>
+        <mesh filename="package://ot2_description/meshes/module_cart.stl" scale="1 1 1"/>
       </geometry>
       <origin xyz="0 0 0" rpy="0 0 0"/>
     </collision>
   </link>
-  <link name="${prefix}pf400_cart">
-    <visual>
-      <origin xyz="-1.592 0.2605 -0.015" rpy="1.5708 0 0"/>
-      <geometry>
-        <mesh filename="package://pf400_description/meshes/pf400_table.STL" scale="0.001 0.001 0.001"/>
-      </geometry>
-      <material name="darkbluegreen"/>
-    </visual>
-    <collision>
-      <geometry>
-        <mesh filename="package://pf400_description/meshes/pf400_table.STL" scale="0.001 0.001 0.001"/>
-      </geometry>
-      <origin xyz="-1.592 0.261 -0.015" rpy="1.5708 0 0"/>
-    </collision>
-  </link>
   <!-- Joints -->
-  <joint name="pf400_cart_to_cart_1" type="fixed">
-    <parent link="${prefix}pf400_cart"/>
-    <child link="${prefix}cart_1"/>
-    <axis xyz="0 0 1"/>
-    <origin xyz="1.0 0.83 0" rpy="0 0 0"/>
-    <limit effort="1000.0" lower="0" upper="0" velocity="0.5"/>
-  </joint>
-  <joint name="pf400_cart_to_cart_2" type="fixed">
-    <parent link="${prefix}pf400_cart"/>
-    <child link="${prefix}cart_2"/>
-    <axis xyz="0 0 1"/>
-    <origin xyz="0.25 0.83 0" rpy="0 0 0"/>
-    <limit effort="1000.0" lower="0" upper="0" velocity="0.5"/>
-  </joint>
-  <joint name="pf400_cart_to_cart_3" type="fixed">
-    <parent link="${prefix}pf400_cart"/>
-    <child link="${prefix}cart_3"/>
-    <axis xyz="0 0 1"/>
-    <origin xyz="-0.50 0.83  0" rpy="0 0 0"/>
-    <limit effort="1000.0" lower="0" upper="0" velocity="0.5"/>
-  </joint>
-  <joint name="pf400_cart_to_cart_4" type="fixed">
-    <parent link="${prefix}pf400_cart"/>
-    <child link="${prefix}cart_4"/>
-    <axis xyz="0 0 1"/>
-    <origin xyz="-1.25 0.83  0" rpy="0 0 0"/>
-    <limit effort="1000.0" lower="0" upper="0" velocity="0.5"/>
-  </joint>
-  <joint name="pf400_cart_to_cart_5" type="fixed">
-    <parent link="${prefix}pf400_cart"/>
-    <child link="${prefix}cart_5"/>
-    <axis xyz="0 0 1"/>
-    <origin xyz="1.00 -0.46 0" rpy="0 0 0"/>
-    <limit effort="1000.0" lower="0" upper="0" velocity="0.5"/>
-  </joint>
-  <joint name="pf400_cart_to_cart_6" type="fixed">
-    <parent link="${prefix}pf400_cart"/>
-    <child link="${prefix}cart_6"/>
-    <axis xyz="0 0 1"/>
-    <origin xyz="0.25 -0.46 0" rpy="0 0 0"/>
-    <limit effort="1000.0" lower="0" upper="0" velocity="0.5"/>
-  </joint>
-  <joint name="pf400_cart_to_cart_7" type="fixed">
-    <parent link="${prefix}pf400_cart"/>
-    <child link="${prefix}cart_7"/>
-    <axis xyz="0 0 1"/>
-    <origin xyz="-0.50 -0.46 0" rpy="0 0 0"/>
-    <limit effort="1000.0" lower="0" upper="0" velocity="0.5"/>
-  </joint>
-  <joint name="pf400_cart_to_cart_8" type="fixed">
-    <parent link="${prefix}pf400_cart"/>
-    <child link="${prefix}cart_8"/>
-    <axis xyz="0 0 1"/>
-    <origin xyz="-1.25 -0.46 0" rpy="0 0 0"/>
-    <limit effort="1000.0" lower="0" upper="0" velocity="0.5"/>
-  </joint>
   </xacro:macro>
 </robot>

Commit message: Have to add the pf400 table to link all the tables

File: ot2_description/urdf/module_carts.urdf.xacro (robot description, xacro)
@@ -3,5 +3,5 @@
   <!-- Links -->
   <xacro:macro name="Module_Carts" params = "prefix">
-  <link name="${prefix}cart_8">
+  <link name="${prefix}cart_1">
     <visual>
       <origin xyz="0 0 0" rpy="0 0 0"/>
@@ -18,5 +18,5 @@
     </collision>
   </link>
-  <link name="${prefix}cart_7">
+  <link name="${prefix}cart_2">
     <visual>
       <origin xyz="0 0 0" rpy="0 0 0"/>
@@ -33,5 +33,5 @@
     </collision>
   </link>
-   <link name="${prefix}cart_4">
+   <link name="${prefix}cart_5">
     <visual>
       <origin xyz="0 0 0" rpy="0 0 0"/>
@@ -48,5 +48,41 @@
     </collision>
   </link>
+  <link name="${prefix}pf400_cart">
+    <visual>
+      <origin xyz="-1.592 0.2605 -0.0" rpy="1.5708 0 0"/>
+      <geometry>
+        <mesh filename="package://pcr_description/meshes/pf400_table.STL" scale="0.001 0.001 0.001"/>
+      </geometry>
+      <material name="darkbluegreen"/>
+    </visual>
+    <collision>
+      <geometry>
+        <mesh filename="package://pcr_description/meshes/pf400_table.STL" scale="0.001 0.001 0.001"/>
+      </geometry>
+      <origin xyz="-1.592 0.261 -0.0" rpy="1.5708 0 0"/>
+    </collision>
+  </link>
   <!-- Joints -->
+  <joint name="pf400_cart_to_cart_1" type="fixed">
+    <parent link="${prefix}pf400_cart"/>
+    <child link="${prefix}cart_1"/>
+    <axis xyz="0 0 1"/>
+    <origin xyz="1.0 0.91 0.005" rpy="0 0 0"/>
+    <limit effort="1000.0" lower="0" upper="0" velocity="0.5"/>
+  </joint>
+  <joint name="pf400_cart_to_cart_2" type="fixed">
+    <parent link="${prefix}pf400_cart"/>
+    <child link="${prefix}cart_2"/>
+    <axis xyz="0 0 1"/>
+    <origin xyz="0.25 0.91 0.005" rpy="0 0 0"/>
+    <limit effort="1000.0" lower="0" upper="0" velocity="0.5"/>
+  </joint>
+  <joint name="pf400_cart_to_cart_5" type="fixed">
+    <parent link="${prefix}pf400_cart"/>
+    <child link="${prefix}cart_5"/>
+    <axis xyz="0 0 1"/>
+    <origin xyz="1.00 -0.54 0.005" rpy="0 0 0"/>
+    <limit effort="1000.0" lower="0" upper="0" velocity="0.5"/>
+  </joint>
   </xacro:macro>
 </robot>
