Commit message: Clean up

File: ot2_description/urdf/OT2.urdf.xacro (robot description, xacro)
@@ -7,11 +7,11 @@
       <origin xyz="0.36 0.94 1.042" rpy="0 0 0"/>
       <geometry>
-        <mesh filename="package://pf400_description/meshes/OT2_base.stl" scale="1 1 1"/>
-      </geometry>
-      <material name="aluminum"/>
-    </visual>
-    <collision>
-      <geometry>
-        <mesh filename="package://pf400_description/meshes/OT2_base.stl" scale="1 1 1"/>
+        <mesh filename="package://ot2_description/meshes/OT2_base.stl" scale="1 1 1"/>
+      </geometry>
+      <material name="aluminum"/>
+    </visual>
+    <collision>
+      <geometry>
+        <mesh filename="package://ot2_description/meshes/OT2_base.stl" scale="1 1 1"/>
       </geometry>
       <origin xyz="0.36 0.94 1.042" rpy="0 0 0"/>
@@ -22,11 +22,11 @@
       <origin xyz="0.36 1.15 1.042" rpy="0 0 0"/>
       <geometry>
-        <mesh filename="package://pf400_description/meshes/OT2_rail.stl" scale="1 1 1"/>
-      </geometry>
-      <material name="aluminum"/>
-    </visual>
-    <collision>
-      <geometry>
-        <mesh filename="package://pf400_description/meshes/OT2_rail.stl" scale="1 1 1"/>
+        <mesh filename="package://ot2_description/meshes/OT2_rail.stl" scale="1 1 1"/>
+      </geometry>
+      <material name="aluminum"/>
+    </visual>
+    <collision>
+      <geometry>
+        <mesh filename="package://ot2_description/meshes/OT2_rail.stl" scale="1 1 1"/>
       </geometry>
       <origin xyz="0.36 1.15 1.042" rpy="0 0 0"/>
@@ -37,11 +37,11 @@
       <origin xyz="0.51 1.15 1.042" rpy="0 0 0"/>
       <geometry>
-        <mesh filename="package://pf400_description/meshes/OT2_pipette_base.stl" scale="1 1 1"/>
-      </geometry>
-      <material name="aluminum"/>
-    </visual>
-    <collision>
-      <geometry>
-        <mesh filename="package://pf400_description/meshes/OT2_pipette_base.stl" scale="1 1 1"/>
+        <mesh filename="package://ot2_description/meshes/OT2_pipette_base.stl" scale="1 1 1"/>
+      </geometry>
+      <material name="aluminum"/>
+    </visual>
+    <collision>
+      <geometry>
+        <mesh filename="package://ot2_description/meshes/OT2_pipette_base.stl" scale="1 1 1"/>
       </geometry>
       <origin xyz="0.51 1.15 1.042" rpy="0 0 0"/>
@@ -52,11 +52,11 @@
       <origin xyz="0.79 0.76 1.27" rpy="1.5708 0 1.5708"/>
       <geometry>
-        <mesh filename="package://pf400_description/meshes/pipette.STL" scale="0.001 0.001 0.001"/>
-      </geometry>
-      <material name="black"/>
-    </visual>
-    <collision>
-      <geometry>
-        <mesh filename="package://pf400_description/meshes/pipette.STL" scale="0.001 0.001 0.001"/>
+        <mesh filename="package://ot2_description/meshes/pipette.STL" scale="0.001 0.001 0.001"/>
+      </geometry>
+      <material name="black"/>
+    </visual>
+    <collision>
+      <geometry>
+        <mesh filename="package://ot2_description/meshes/pipette.STL" scale="0.001 0.001 0.001"/>
       </geometry>
       <origin xyz="0.79 0.76 1.27" rpy="1.5708 0 1.5708"/>
@@ -67,11 +67,11 @@
       <origin xyz="0.51 1.15 1.042" rpy="0 0 0"/>
       <geometry>
-        <mesh filename="package://pf400_description/meshes/OT2_8ch_pipette.stl" scale="1 1 1"/>
-      </geometry>
-      <material name="black"/>
-    </visual>
-    <collision>
-      <geometry>
-        <mesh filename="package://pf400_description/meshes/OT2_8ch_pipette.stl" scale="1 1 1"/>
+        <mesh filename="package://ot2_description/meshes/OT2_8ch_pipette.stl" scale="1 1 1"/>
+      </geometry>
+      <material name="black"/>
+    </visual>
+    <collision>
+      <geometry>
+        <mesh filename="package://ot2_description/meshes/OT2_8ch_pipette.stl" scale="1 1 1"/>
       </geometry>
       <origin xyz="0.51 1.15 1.042" rpy="0 0 0"/>
@@ -82,11 +82,11 @@
       <origin xyz="0.36 0.94 1.042" rpy="0 0 0"/>
       <geometry>
-        <mesh filename="package://pf400_description/meshes/OT2_base.stl" scale="1 1 1"/>
-      </geometry>
-      <material name="aluminum"/>
-    </visual>
-    <collision>
-      <geometry>
-        <mesh filename="package://pf400_description/meshes/OT2_base.stl" scale="1 1 1"/>
+        <mesh filename="package://ot2_description/meshes/OT2_base.stl" scale="1 1 1"/>
+      </geometry>
+      <material name="aluminum"/>
+    </visual>
+    <collision>
+      <geometry>
+        <mesh filename="package://ot2_description/meshes/OT2_base.stl" scale="1 1 1"/>
       </geometry>
       <origin xyz="0.36 0.94 1.042" rpy="0 0 0"/>
@@ -97,11 +97,11 @@
       <origin xyz="0.36 1.15 1.042" rpy="0 0 0"/>
       <geometry>
-        <mesh filename="package://pf400_description/meshes/OT2_rail.stl" scale="1 1 1"/>
-      </geometry>
-      <material name="aluminum"/>
-    </visual>
-    <collision>
-      <geometry>
-        <mesh filename="package://pf400_description/meshes/OT2_rail.stl" scale="1 1 1"/>
+        <mesh filename="package://ot2_description/meshes/OT2_rail.stl" scale="1 1 1"/>
+      </geometry>
+      <material name="aluminum"/>
+    </visual>
+    <collision>
+      <geometry>
+        <mesh filename="package://ot2_description/meshes/OT2_rail.stl" scale="1 1 1"/>
       </geometry>
       <origin xyz="0.36 1.15 1.042" rpy="0 0 0"/>
@@ -112,11 +112,11 @@
       <origin xyz="0.51 1.15 1.042" rpy="0 0 0"/>
       <geometry>
-        <mesh filename="package://pf400_description/meshes/OT2_pipette_base.stl" scale="1 1 1"/>
-      </geometry>
-      <material name="aluminum"/>
-    </visual>
-    <collision>
-      <geometry>
-        <mesh filename="package://pf400_description/meshes/OT2_pipette_base.stl" scale="1 1 1"/>
+        <mesh filename="package://ot2_description/meshes/OT2_pipette_base.stl" scale="1 1 1"/>
+      </geometry>
+      <material name="aluminum"/>
+    </visual>
+    <collision>
+      <geometry>
+        <mesh filename="package://ot2_description/meshes/OT2_pipette_base.stl" scale="1 1 1"/>
       </geometry>
       <origin xyz="0.51 1.15 1.042" rpy="0 0 0"/>
@@ -127,11 +127,11 @@
       <origin xyz="0.79 0.76 1.27" rpy="1.5708 0 1.5708"/>
       <geometry>
-        <mesh filename="package://pf400_description/meshes/pipette.STL" scale="0.001 0.001 0.001"/>
-      </geometry>
-      <material name="black"/>
-    </visual>
-    <collision>
-      <geometry>
-        <mesh filename="package://pf400_description/meshes/pipette.STL" scale="0.001 0.001 0.001"/>
+        <mesh filename="package://ot2_description/meshes/pipette.STL" scale="0.001 0.001 0.001"/>
+      </geometry>
+      <material name="black"/>
+    </visual>
+    <collision>
+      <geometry>
+        <mesh filename="package://ot2_description/meshes/pipette.STL" scale="0.001 0.001 0.001"/>
       </geometry>
       <origin xyz="0.79 0.76 1.27" rpy="1.5708 0 1.5708"/>
@@ -142,11 +142,11 @@
       <origin xyz="0.51 1.15 1.042" rpy="0 0 0"/>
       <geometry>
-        <mesh filename="package://pf400_description/meshes/OT2_8ch_pipette.stl" scale="1 1 1"/>
-      </geometry>
-      <material name="black"/>
-    </visual>
-    <collision>
-      <geometry>
-        <mesh filename="package://pf400_description/meshes/OT2_8ch_pipette.stl" scale="1 1 1"/>
+        <mesh filename="package://ot2_description/meshes/OT2_8ch_pipette.stl" scale="1 1 1"/>
+      </geometry>
+      <material name="black"/>
+    </visual>
+    <collision>
+      <geometry>
+        <mesh filename="package://ot2_description/meshes/OT2_8ch_pipette.stl" scale="1 1 1"/>
       </geometry>
       <origin xyz="0.51 1.15 1.042" rpy="0 0 0"/>
@@ -154,5 +154,5 @@
   </link>
   <!-- Joints -->
-  <joint name="OT2_1_Pipette_Joint1_alpha" type="fixed">
+  <joint name="OT2_1_Pipette_Joint1_alpha" type="prismatic">
     <parent link="${prefix}OT2_alpha"/>
     <child link="${prefix}OT2_pipette_rail_alpha"/>
@@ -161,5 +161,5 @@
     <limit effort="1000.0" lower="0" upper="0.3" velocity="0.5"/>
   </joint>
-  <joint name="OT2_1_Pipette_Joint2_alpha" type="fixed">
+  <joint name="OT2_1_Pipette_Joint2_alpha" type="prismatic">
     <parent link="${prefix}OT2_pipette_rail_alpha"/>
     <child link="${prefix}OT2_pipette_base_alpha"/>
@@ -168,5 +168,5 @@
     <limit effort="1000.0" lower="0" upper="0.3" velocity="0.5"/>
   </joint>
-  <joint name="OT2_1_Single_Pipette_alpha" type="fixed">
+  <joint name="OT2_1_Single_Pipette_alpha" type="prismatic">
     <parent link="${prefix}OT2_pipette_base_alpha"/>
     <child link="${prefix}OT2_single_pipette_alpha"/>
@@ -175,5 +175,5 @@
     <limit effort="1000.0" lower="0" upper="0.18" velocity="0.5"/>
   </joint>
-  <joint name="OT2_1_8_Channel_Pipette_alpha" type="fixed">
+  <joint name="OT2_1_8_Channel_Pipette_alpha" type="prismatic">
     <parent link="${prefix}OT2_pipette_base_alpha"/>
     <child link="${prefix}OT2_8_channel_pipette_alpha"/>
@@ -182,5 +182,5 @@
     <limit effort="1000.0" lower="0" upper="0.18" velocity="0.5"/>
   </joint>
-  <joint name="OT2_1_Pipette_Joint1_betha" type="fixed">
+  <joint name="OT2_1_Pipette_Joint1_betha" type="prismatic">
     <parent link="${prefix}OT2_betha"/>
     <child link="${prefix}OT2_pipette_rail_betha"/>
@@ -189,5 +189,5 @@
     <limit effort="1000.0" lower="0" upper="0.3" velocity="0.5"/>
   </joint>
-  <joint name="OT2_1_Pipette_Joint2_betha" type="fixed">
+  <joint name="OT2_1_Pipette_Joint2_betha" type="prismatic">
     <parent link="${prefix}OT2_pipette_rail_betha"/>
     <child link="${prefix}OT2_pipette_base_betha"/>
@@ -196,5 +196,5 @@
     <limit effort="1000.0" lower="0" upper="0.3" velocity="0.5"/>
   </joint>
-  <joint name="OT2_1_Single_Pipette_betha" type="fixed">
+  <joint name="OT2_1_Single_Pipette_betha" type="prismatic">
     <parent link="${prefix}OT2_pipette_base_betha"/>
     <child link="${prefix}OT2_single_pipette_betha"/>
@@ -203,5 +203,5 @@
     <limit effort="1000.0" lower="0" upper="0.18" velocity="0.5"/>
   </joint>
-  <joint name="OT2_1_8_Channel_Pipette_betha" type="fixed">
+  <joint name="OT2_1_8_Channel_Pipette_betha" type="prismatic">
     <parent link="${prefix}OT2_pipette_base_betha"/>
     <child link="${prefix}OT2_8_channel_pipette_betha"/>

Commit message: Fixing mesh import

File: ot2_description/urdf/OT2.urdf.xacro (robot description, xacro)
@@ -37,11 +37,11 @@
       <origin xyz="0.51 1.15 1.042" rpy="0 0 0"/>
       <geometry>
-        <mesh filename="package://ot2_description/meshes/OT2_pipette_base.stl" scale="1 1 1"/>
-      </geometry>
-      <material name="aluminum"/>
-    </visual>
-    <collision>
-      <geometry>
-        <mesh filename="package://ot2_description/meshes/OT2_pipette_base.stl" scale="1 1 1"/>
+        <mesh filename="package://ot2_description/meshes/OT2_pipette_base.STL" scale="1 1 1"/>
+      </geometry>
+      <material name="aluminum"/>
+    </visual>
+    <collision>
+      <geometry>
+        <mesh filename="package://ot2_description/meshes/OT2_pipette_base.STL" scale="1 1 1"/>
       </geometry>
       <origin xyz="0.51 1.15 1.042" rpy="0 0 0"/>
@@ -112,11 +112,11 @@
       <origin xyz="0.51 1.15 1.042" rpy="0 0 0"/>
       <geometry>
-        <mesh filename="package://ot2_description/meshes/OT2_pipette_base.stl" scale="1 1 1"/>
-      </geometry>
-      <material name="aluminum"/>
-    </visual>
-    <collision>
-      <geometry>
-        <mesh filename="package://ot2_description/meshes/OT2_pipette_base.stl" scale="1 1 1"/>
+        <mesh filename="package://ot2_description/meshes/OT2_pipette_base.STL" scale="1 1 1"/>
+      </geometry>
+      <material name="aluminum"/>
+    </visual>
+    <collision>
+      <geometry>
+        <mesh filename="package://ot2_description/meshes/OT2_pipette_base.STL" scale="1 1 1"/>
       </geometry>
       <origin xyz="0.51 1.15 1.042" rpy="0 0 0"/>

Commit message: Adding OT2 gamma

File: ot2_description/urdf/OT2.urdf.xacro (robot description, xacro)
@@ -153,4 +153,79 @@
     </collision>
   </link>
+   <link name="${prefix}OT2_gamma">
+    <visual>
+      <origin xyz="0.36 0.94 1.042" rpy="0 0 0"/>
+      <geometry>
+        <mesh filename="package://ot2_description/meshes/OT2_base.stl" scale="1 1 1"/>
+      </geometry>
+      <material name="aluminum"/>
+    </visual>
+    <collision>
+      <geometry>
+        <mesh filename="package://ot2_description/meshes/OT2_base.stl" scale="1 1 1"/>
+      </geometry>
+      <origin xyz="0.36 0.94 1.042" rpy="0 0 0"/>
+    </collision>
+  </link>
+  <link name="${prefix}OT2_pipette_rail_gamma">
+    <visual>
+      <origin xyz="0.36 1.15 1.042" rpy="0 0 0"/>
+      <geometry>
+        <mesh filename="package://ot2_description/meshes/OT2_rail.stl" scale="1 1 1"/>
+      </geometry>
+      <material name="aluminum"/>
+    </visual>
+    <collision>
+      <geometry>
+        <mesh filename="package://ot2_description/meshes/OT2_rail.stl" scale="1 1 1"/>
+      </geometry>
+      <origin xyz="0.36 1.15 1.042" rpy="0 0 0"/>
+    </collision>
+  </link>
+  <link name="${prefix}OT2_pipette_base_gamma">
+    <visual>
+      <origin xyz="0.51 1.15 1.042" rpy="0 0 0"/>
+      <geometry>
+        <mesh filename="package://ot2_description/meshes/OT2_pipette_base.STL" scale="1 1 1"/>
+      </geometry>
+      <material name="aluminum"/>
+    </visual>
+    <collision>
+      <geometry>
+        <mesh filename="package://ot2_description/meshes/OT2_pipette_base.STL" scale="1 1 1"/>
+      </geometry>
+      <origin xyz="0.51 1.15 1.042" rpy="0 0 0"/>
+    </collision>
+  </link>
+  <link name="${prefix}OT2_single_pipette_gamma">
+    <visual>
+      <origin xyz="0.79 0.76 1.27" rpy="1.5708 0 1.5708"/>
+      <geometry>
+        <mesh filename="package://ot2_description/meshes/pipette.STL" scale="0.001 0.001 0.001"/>
+      </geometry>
+      <material name="black"/>
+    </visual>
+    <collision>
+      <geometry>
+        <mesh filename="package://ot2_description/meshes/pipette.STL" scale="0.001 0.001 0.001"/>
+      </geometry>
+      <origin xyz="0.79 0.76 1.27" rpy="1.5708 0 1.5708"/>
+    </collision>
+  </link>
+  <link name="${prefix}OT2_8_channel_pipette_gamma">
+    <visual>
+      <origin xyz="0.51 1.15 1.042" rpy="0 0 0"/>
+      <geometry>
+        <mesh filename="package://ot2_description/meshes/OT2_8ch_pipette.stl" scale="1 1 1"/>
+      </geometry>
+      <material name="black"/>
+    </visual>
+    <collision>
+      <geometry>
+        <mesh filename="package://ot2_description/meshes/OT2_8ch_pipette.stl" scale="1 1 1"/>
+      </geometry>
+      <origin xyz="0.51 1.15 1.042" rpy="0 0 0"/>
+    </collision>
+  </link>
   <!-- Joints -->
   <joint name="OT2_1_Pipette_Joint1_alpha" type="prismatic">
@@ -210,4 +285,32 @@
     <limit effort="1000.0" lower="0" upper="0.18" velocity="0.5"/>
   </joint>
+    <joint name="OT2_1_Pipette_Joint1_gamma" type="prismatic">
+    <parent link="${prefix}OT2_gamma"/>
+    <child link="${prefix}OT2_pipette_rail_gamma"/>
+    <axis xyz="0 -1 0"/>
+    <origin xyz="0 0 0" rpy="0 0 0"/>
+    <limit effort="1000.0" lower="0" upper="0.3" velocity="0.5"/>
+  </joint>
+  <joint name="OT2_1_Pipette_Joint2_gamma" type="prismatic">
+    <parent link="${prefix}OT2_pipette_rail_gamma"/>
+    <child link="${prefix}OT2_pipette_base_gamma"/>
+    <axis xyz="-1 0 0"/>
+    <origin xyz="0 0 0" rpy="0 0 0"/>
+    <limit effort="1000.0" lower="0" upper="0.3" velocity="0.5"/>
+  </joint>
+  <joint name="OT2_1_Single_Pipette_gamma" type="prismatic">
+    <parent link="${prefix}OT2_pipette_base_gamma"/>
+    <child link="${prefix}OT2_single_pipette_gamma"/>
+    <axis xyz="0 0 -1"/>
+    <origin xyz="0 0 0" rpy="0 0 0"/>
+    <limit effort="1000.0" lower="0" upper="0.18" velocity="0.5"/>
+  </joint>
+  <joint name="OT2_1_8_Channel_Pipette_gamma" type="prismatic">
+    <parent link="${prefix}OT2_pipette_base_gamma"/>
+    <child link="${prefix}OT2_8_channel_pipette_gamma"/>
+    <axis xyz="0 0 -1"/>
+    <origin xyz="0 0 0" rpy="0 0 0"/>
+    <limit effort="1000.0" lower="0" upper="0.18" velocity="0.5"/>
+  </joint>
   </xacro:macro>
 </robot>

File: ot2_description/urdf/OT2_robot.xacro (robot description, xacro)
@@ -23,3 +23,10 @@
     <limit effort="1000.0" lower="0" upper="0" velocity="0.5"/>
   </joint>
+  <joint name="OT2_gamma" type="fixed">
+    <parent link="module_carts/cart_4"/>
+    <child link="ot2/OT2_gamma"/>
+    <axis xyz="0 0 0"/>
+    <origin xyz="0.825 0.47 0" rpy="0 0 3.1416"/>
+    <limit effort="1000.0" lower="0" upper="0" velocity="0.5"/>
+  </joint>
 </robot>

Commit message: Clean up

File: ot2_description/urdf/OT2.urdf.xacro (robot description, xacro)
@@ -285,5 +285,5 @@
     <limit effort="1000.0" lower="0" upper="0.18" velocity="0.5"/>
   </joint>
-    <joint name="OT2_1_Pipette_Joint1_gamma" type="prismatic">
+  <joint name="OT2_1_Pipette_Joint1_gamma" type="prismatic">
     <parent link="${prefix}OT2_gamma"/>
     <child link="${prefix}OT2_pipette_rail_gamma"/>

Commit message: Renaming the joints

File: ot2_description/urdf/OT2.urdf.xacro (robot description, xacro)
@@ -229,5 +229,5 @@
   </link>
   <!-- Joints -->
-  <joint name="OT2_1_Pipette_Joint1_alpha" type="prismatic">
+  <joint name="OT2_Alpha_Pipette_Joint1" type="prismatic">
     <parent link="${prefix}OT2_alpha"/>
     <child link="${prefix}OT2_pipette_rail_alpha"/>
@@ -236,5 +236,5 @@
     <limit effort="1000.0" lower="0" upper="0.3" velocity="0.5"/>
   </joint>
-  <joint name="OT2_1_Pipette_Joint2_alpha" type="prismatic">
+  <joint name="OT2_Alpha_Pipette_Joint2" type="prismatic">
     <parent link="${prefix}OT2_pipette_rail_alpha"/>
     <child link="${prefix}OT2_pipette_base_alpha"/>
@@ -243,5 +243,5 @@
     <limit effort="1000.0" lower="0" upper="0.3" velocity="0.5"/>
   </joint>
-  <joint name="OT2_1_Single_Pipette_alpha" type="prismatic">
+  <joint name="OT2_Alpha_Single_Pipette" type="prismatic">
     <parent link="${prefix}OT2_pipette_base_alpha"/>
     <child link="${prefix}OT2_single_pipette_alpha"/>
@@ -250,5 +250,5 @@
     <limit effort="1000.0" lower="0" upper="0.18" velocity="0.5"/>
   </joint>
-  <joint name="OT2_1_8_Channel_Pipette_alpha" type="prismatic">
+  <joint name="OT2_Alpha_8_Channel_Pipette" type="prismatic">
     <parent link="${prefix}OT2_pipette_base_alpha"/>
     <child link="${prefix}OT2_8_channel_pipette_alpha"/>
@@ -257,5 +257,5 @@
     <limit effort="1000.0" lower="0" upper="0.18" velocity="0.5"/>
   </joint>
-  <joint name="OT2_1_Pipette_Joint1_betha" type="prismatic">
+  <joint name="OT2_Betha_Pipette_Joint1" type="prismatic">
     <parent link="${prefix}OT2_betha"/>
     <child link="${prefix}OT2_pipette_rail_betha"/>
@@ -264,5 +264,5 @@
     <limit effort="1000.0" lower="0" upper="0.3" velocity="0.5"/>
   </joint>
-  <joint name="OT2_1_Pipette_Joint2_betha" type="prismatic">
+  <joint name="OT2_Betha_Pipette_Joint2" type="prismatic">
     <parent link="${prefix}OT2_pipette_rail_betha"/>
     <child link="${prefix}OT2_pipette_base_betha"/>
@@ -271,5 +271,5 @@
     <limit effort="1000.0" lower="0" upper="0.3" velocity="0.5"/>
   </joint>
-  <joint name="OT2_1_Single_Pipette_betha" type="prismatic">
+  <joint name="OT2_Betha_Single_Pipette" type="prismatic">
     <parent link="${prefix}OT2_pipette_base_betha"/>
     <child link="${prefix}OT2_single_pipette_betha"/>
@@ -278,5 +278,5 @@
     <limit effort="1000.0" lower="0" upper="0.18" velocity="0.5"/>
   </joint>
-  <joint name="OT2_1_8_Channel_Pipette_betha" type="prismatic">
+  <joint name="OT2_Betha_8_Channel_Pipette" type="prismatic">
     <parent link="${prefix}OT2_pipette_base_betha"/>
     <child link="${prefix}OT2_8_channel_pipette_betha"/>
@@ -285,5 +285,5 @@
     <limit effort="1000.0" lower="0" upper="0.18" velocity="0.5"/>
   </joint>
-  <joint name="OT2_1_Pipette_Joint1_gamma" type="prismatic">
+  <joint name="OT2_Gamma_Pipette_Joint1" type="prismatic">
     <parent link="${prefix}OT2_gamma"/>
     <child link="${prefix}OT2_pipette_rail_gamma"/>
@@ -292,5 +292,5 @@
     <limit effort="1000.0" lower="0" upper="0.3" velocity="0.5"/>
   </joint>
-  <joint name="OT2_1_Pipette_Joint2_gamma" type="prismatic">
+  <joint name="OT2_Gamma_Pipette_Joint2" type="prismatic">
     <parent link="${prefix}OT2_pipette_rail_gamma"/>
     <child link="${prefix}OT2_pipette_base_gamma"/>
@@ -299,5 +299,5 @@
     <limit effort="1000.0" lower="0" upper="0.3" velocity="0.5"/>
   </joint>
-  <joint name="OT2_1_Single_Pipette_gamma" type="prismatic">
+  <joint name="OT2_Gamma_Single_Pipette" type="prismatic">
     <parent link="${prefix}OT2_pipette_base_gamma"/>
     <child link="${prefix}OT2_single_pipette_gamma"/>
@@ -306,5 +306,5 @@
     <limit effort="1000.0" lower="0" upper="0.18" velocity="0.5"/>
   </joint>
-  <joint name="OT2_1_8_Channel_Pipette_gamma" type="prismatic">
+  <joint name="OT2_Gamma_8_Channel_Pipette" type="prismatic">
     <parent link="${prefix}OT2_pipette_base_gamma"/>
     <child link="${prefix}OT2_8_channel_pipette_gamma"/>
